File: M.O.L.D Circuit Diagram (KiCad)/M.O.L.D Circuit Diagram.kicad_sch (KiCad schematic)
At the start: 10 parts, among them M1 Fan, Q1 PN2222A, SW1 SW_DPDT_x2, U1 DHT11, U3 LCD_I2C

Commit message: Humidity Threshold Change
Other:
- title: (none) -> Arduino Mold Prevention System
- moved on the sheet: A1, D1, D2, M1, Q1, R1, R2, SW1A, U1, U3
